File: PCB/blueprintpcb1.kicad_pcb (KiCad board)
At the start: 2 copper layers, 100 x 56 mm, 18 parts, among them J1 Conn_01x04_Pin, SW1 SW_Push, SW2 SW_Push, SW3 SW_Push, SW4 SW_Push, SW5 RotaryEncoder_Switch, SW6 SW_Push, U1 XIAO-RP2040-DIP

Commit message: update pcb
Parts:
- D1, D2: footprint LED_SMD:LED_SK6812MINI_PLCC4_3.5x3.5mm_P1.75mm -> decor:MX_SK6812MINI-E_REV
- moved D1 17.7 mm to (211.3, 139.6), turned to 180 degrees
- moved D2 16.5 mm to (230.3, 139.5), turned to 180 degrees
- moved G*** 5.70 mm to (220.5, 117.5)
Routing:
- net Net-(D1-DIN): track 18.4 -> 15.3 mm
- net GND: track 115.1 -> 118.1 mm, vias 3 -> 2
- net LED: track 31.4 -> 28.7 mm, vias 2 -> 1
- net +5V: track 46.2 -> 45.6 mm, vias 2 -> 1
