File: PCB/blueprintpcb1.kicad_sch (KiCad schematic)
At the start: 7 parts, among them SW1 SW_Push, SW2 SW_Push, SW3 SW_Push, SW4 SW_Push, U1 XIAO-RP2040-DIP

Commit message: ver2
Parts:
- added D3, D4, D5, D6, D7, D8: D_Small, Diode_THT:D_DO-35_SOD27_P7.62mm_Horizontal, symbol Device:D_Small
- added J1: Conn_01x04_Pin, Connector_PinHeader_2.54mm:PinHeader_1x04_P2.54mm_Vertical, symbol Connector:Conn_01x04_Pin
- added SW5: RotaryEncoder_Switch, Rotary_Encoder:RotaryEncoder_Alps_EC11E-Switch_Vertical_H20mm, symbol Device:RotaryEncoder_Switch
- added SW6: SW_Push, Button_Switch_Keyboard:SW_Cherry_MX_1.00u_PCB, symbol Switch:SW_Push
- U1: footprint OPL_kicad_library:XIAO-RP2040-DIP -> Seeed Studio XIAO Series Library:XIAO-RP2040-DIP
Connections:
- net GND: now also J1.4 (Pin_4), SW5.C; no longer SW1.1, SW2.1, SW3.1, SW4.1
- net at SW1.2: now also D3.2 (A); no longer U1.11 (GPIO3/MOSI)
- net LED: now reaches D2.3 (DIN)
- net LED: now also U1.11 (GPIO3/MOSI); no longer U1.5 (GPIO6/SDA)
- net COL0: now reaches U1.1 (GPIO26/ADC0/A0)
- net COL0: now also SW1.1, SW2.1
- net at SW2.2: now also D5.2 (A); no longer U1.10 (GPIO4/MISO)
- net COL1: now reaches U1.2 (GPIO27/ADC1/A1)
- net COL1: now also SW3.1, SW6.1
- net ROW0: now reaches U1.3 (GPIO28/ADC2/A2)
- net ROW0: now also D3.1 (K), D4.1 (K), D8.1 (K)
- net ROW1: now reaches U1.4 (GPIO29/ADC3/A3)
- net ROW1: now also D5.1 (K), D6.1 (K), D7.1 (K)
- net SCL: now reaches U1.6 (GPIO7/SCL)
- net SCL: now also J1.2 (Pin_2)
- net at SW4.2: now also D7.2 (A); no longer U1.8 (GPIO1/RX)
- net at SW3.2: now also D6.2 (A); no longer U1.9 (GPIO2/SCK)
- new net: D4.2 (A), SW6.2
- new net COL2: SW4.1, SW5.S2, U1.10 (GPIO4/MISO)
- new net EC11A: SW5.A, U1.9 (GPIO2/SCK)
- new net EC11B: SW5.B, U1.8 (GPIO1/RX)
- new net EC11SWA: D8.2 (A), SW5.S1
- new net SDA: J1.1 (Pin_1), U1.5 (GPIO6/SDA)
- new net VCC: J1.3 (Pin_3)
- no-connect marks 8 -> 2
Other:
- note added: "LED"
- note added: "MATRIX"
- note added: "OLED"
- note added: "ROTARY ENCODER"
- moved on the sheet: D1, D2, SW1, SW2, SW3, SW4, U1

Commit message: update pcb
Parts:
- D1, D2: footprint LED_SMD:LED_SK6812MINI_PLCC4_3.5x3.5mm_P1.75mm -> decor:MX_SK6812MINI-E_REV
Changed lines of the file:
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@@
 			)
 		)
-		(property "Footprint" "LED_SMD:LED_SK6812MINI_PLCC4_3.5x3.5mm_P1.75mm"
+		(property "Footprint" "decor:MX_SK6812MINI-E_REV"
 			(at 140.97 41.91 0)
 			(effects
@@
 			)
 		)
-		(property "Footprint" "LED_SMD:LED_SK6812MINI_PLCC4_3.5x3.5mm_P1.75mm"
+		(property "Footprint" "decor:MX_SK6812MINI-E_REV"
 			(at 177.8 41.91 0)
 			(effects
